Commit message: Align RobotLab Thunder inertials with standalone asset
The standalone thunder_v3_assets repository is the canonical source for the corrected Thunder v3 dynamics. The RobotLab copy now matches that primary URDF exactly while keeping the local file name selected for the training asset config, so the GitHub asset repository and RobotLab branch no longer carry different wheel/foot masses or inertial tensors.

Constraint: thunder_v3_assets master defines cad-2026-05-02-symmetric-wheel as the authoritative asset version
Rejected: Keep the raw-CAD inertial copy in RobotLab | it diverged from the standalone asset's corrected wheel/foot mass and symmetry fixes
Confidence: high
Scope-risk: narrow
Directive: When updating Thunder inertials, keep RobotLab's copied URDF synchronized with Kitjesen/thunder_v3_assets unless a training-specific fork is explicitly documented
Tested: XML parse, 21 links, 20 joints, 48.79163 kg total mass, mesh path existence, exact byte match with standalone urdf/thunder_v3.urdf, py_compile thunder.py, git diff --check
Not-tested: IsaacLab runtime scene load or policy rollout

File: robot_lab/data/Robots/thunder_v3_assets/urdf/thunder_v3_cad_inertia.urdf (robot description, URDF)
Before this commit: robot thunder_v3, 21 links, 20 joints
Links:
- link FL_foot: mass 0.32377 -> 1.40377
- link FL_hip: mass 1.66356 -> 1.78126
- link FL_thigh: mass 2.41000 -> 2.40982
- link FR_foot: mass 0.32377 -> 1.40377
- link FR_hip: mass 1.66356 -> 1.78126
- link FR_thigh: mass 2.41000 -> 2.40982
- link RL_foot: mass 0.32377 -> 1.40377
- link RL_hip: mass 1.66356 -> 1.78126
- link RL_thigh: mass 2.41000 -> 2.40982
- link RR_foot: mass 0.32377 -> 1.40377
- link RR_hip: mass 1.66356 -> 1.78126
- link RR_thigh: mass 2.41000 -> 2.40982
Joints:
- joint FL_calf_joint: limit lower=-3.14 upper=0 effort=0 velocity=0 -> lower=-3.14 upper=0 effort=120 velocity=17.48
- joint FL_hip_joint: limit lower=-0.41 upper=0.41 effort=0 velocity=0 -> lower=-0.41 upper=0.41 effort=120 velocity=17.48
- joint FL_thigh_joint: limit lower=0 upper=3.14 effort=0 velocity=0 -> lower=0 upper=3.14 effort=120 velocity=17.48
- joint FR_calf_joint: limit lower=0 upper=3.14 effort=0 velocity=0 -> lower=0 upper=3.14 effort=120 velocity=17.48
- joint FR_hip_joint: limit lower=-0.41 upper=0.41 effort=0 velocity=0 -> lower=-0.41 upper=0.41 effort=120 velocity=17.48
- joint FR_thigh_joint: limit lower=-3.14 upper=0 effort=0 velocity=0 -> lower=-3.14 upper=0 effort=120 velocity=17.48
- joint RL_calf_joint: limit lower=0 upper=6.28 effort=0 velocity=0 -> lower=0 upper=3.14 effort=120 velocity=17.48
- joint RL_hip_joint: limit lower=-0.41 upper=0.41 effort=0 velocity=0 -> lower=-0.41 upper=0.41 effort=120 velocity=17.48
- joint RL_thigh_joint: limit lower=-3.14 upper=0 effort=0 velocity=0 -> lower=-3.14 upper=0 effort=120 velocity=17.48
- joint RR_calf_joint: limit lower=-6.28 upper=0 effort=0 velocity=0 -> lower=-3.14 upper=0 effort=120 velocity=17.48
- joint RR_hip_joint: limit lower=-0.41 upper=0.41 effort=0 velocity=0 -> lower=-0.41 upper=0.41 effort=120 velocity=17.48
- joint RR_thigh_joint: limit lower=0 upper=3.14 effort=0 velocity=0 -> lower=0 upper=3.14 effort=120 velocity=17.48
