Commit message: Keep RobotLab Thunder asset on 0131 limits
RobotLab should consume the same training-safe Thunder v3 asset as the standalone asset repository. This sync replaces the stale raw-CAD style limits and zero motor metadata with the CAD-inertia asset using legacy 0131 position limits.

Constraint: Match the standalone thunder_v3_assets URDF used on the training machine

Constraint: Preserve continuous wheel joints with no limit tags

Rejected: Patch only the changed limit fields | thunder_v3.urdf also contained stale zero effort/velocity metadata and older inertials

Confidence: high

Scope-risk: moderate

Directive: Keep thunder_v3.urdf and thunder_v3_cad_inertia.urdf synchronized for this asset

Tested: Parsed both RobotLab URDFs; verified hips [-0.4,0.4], rear calves [-3.14,3.14], foot joints without limit tags, effort 120, velocity 17.48

Not-tested: Restarted training from the committed RobotLab sync branch

File: robot_lab/data/Robots/thunder_v3_assets/urdf/thunder_v3.urdf (robot description, URDF)
Before this commit: robot thunder_v3, 21 links, 20 joints
Links:
- link FL_foot: mass 0.32377 -> 1.40377
- link FR_foot: mass 0.32377 -> 1.40377
- link RL_foot: mass 0.32377 -> 1.40377
- link RR_foot: mass 0.32377 -> 1.40377
Joints:
- joint FL_calf_joint: limit lower=-3.14 upper=0 effort=0 velocity=0 -> lower=-3.14 upper=0 effort=120 velocity=17.48
- joint FL_hip_joint: limit lower=-0.41 upper=0.41 effort=0 velocity=0 -> lower=-0.4 upper=0.4 effort=120 velocity=17.48
- joint FL_thigh_joint: limit lower=0 upper=3.14 effort=0 velocity=0 -> lower=0 upper=3.14 effort=120 velocity=17.48
- joint FR_calf_joint: limit lower=0 upper=3.14 effort=0 velocity=0 -> lower=0 upper=3.14 effort=120 velocity=17.48
- joint FR_hip_joint: limit lower=-0.41 upper=0.41 effort=0 velocity=0 -> lower=-0.4 upper=0.4 effort=120 velocity=17.48
- joint FR_thigh_joint: limit lower=-3.14 upper=0 effort=0 velocity=0 -> lower=-3.14 upper=0 effort=120 velocity=17.48
- joint RL_calf_joint: limit lower=0 upper=6.28 effort=0 velocity=0 -> lower=-3.14 upper=3.14 effort=120 velocity=17.48
- joint RL_hip_joint: limit lower=-0.41 upper=0.41 effort=0 velocity=0 -> lower=-0.4 upper=0.4 effort=120 velocity=17.48
- joint RL_thigh_joint: limit lower=-3.14 upper=0 effort=0 velocity=0 -> lower=-3.14 upper=0 effort=120 velocity=17.48
- joint RR_calf_joint: limit lower=-6.28 upper=0 effort=0 velocity=0 -> lower=-3.14 upper=3.14 effort=120 velocity=17.48
- joint RR_hip_joint: limit lower=-0.41 upper=0.41 effort=0 velocity=0 -> lower=-0.4 upper=0.4 effort=120 velocity=17.48
- joint RR_thigh_joint: limit lower=0 upper=3.14 effort=0 velocity=0 -> lower=0 upper=3.14 effort=120 velocity=17.48

File: robot_lab/data/Robots/thunder_v3_assets/urdf/thunder_v3_cad_inertia.urdf (robot description, URDF)
Before this commit: robot thunder_v3, 21 links, 20 joints
Joints:
- joint FL_hip_joint: limit lower=-0.41 upper=0.41 effort=120 velocity=17.48 -> lower=-0.4 upper=0.4 effort=120 velocity=17.48
- joint FR_hip_joint: limit lower=-0.41 upper=0.41 effort=120 velocity=17.48 -> lower=-0.4 upper=0.4 effort=120 velocity=17.48
- joint RL_calf_joint: limit lower=0 upper=3.14 effort=120 velocity=17.48 -> lower=-3.14 upper=3.14 effort=120 velocity=17.48
- joint RL_hip_joint: limit lower=-0.41 upper=0.41 effort=120 velocity=17.48 -> lower=-0.4 upper=0.4 effort=120 velocity=17.48
- joint RR_calf_joint: limit lower=-3.14 upper=0 effort=120 velocity=17.48 -> lower=-3.14 upper=3.14 effort=120 velocity=17.48
- joint RR_hip_joint: limit lower=-0.41 upper=0.41 effort=120 velocity=17.48 -> lower=-0.4 upper=0.4 effort=120 velocity=17.48
